Commit message: 有bug，gazebo一半

File: src/wmq_description/urdf/wmqbot/base.urdf.xacro (robot description, xacro)
@@ -27,5 +27,5 @@
             <xacro:cylinder_inertia m="1.0" r="${radius}" h="${length}" />
         </link>
-        <joint name="joint_name" type="fixed">
+        <joint name="base_footprint_joint" type="fixed">
             <origin xyz="0.0 0.0 ${length/2.0+0.032-0.01}" rpy="0.0 0.0 0.0"/>
             <parent link="base_footprint"/>
