Commit message: xacro模型搭建完成

File: src/wmq_description/urdf/wmqbot/actuator/caster.urdf.xacro (robot description, xacro)
@@ -1,4 +1,5 @@
 <?xml version="1.0"?>
 <robot xmlns:xacro="http://www.ros.org/wiki/xacro">
+    <xacro:include filename="$(find wmq_description)/urdf/wmqbot/common_inertia.xacro" />
     <xacro:macro name="caster_xacro" params="caster_name xyz">
         <!-- 机器人的身体部分 -->
@@ -15,4 +16,14 @@
                 </material>
             </visual>
+            <collision>
+                <origin xyz="0.0 0.0 0.0" rpy="0.0 0.0 0.0"/>
+                <geometry>
+                    <sphere radius="0.016"/>
+                </geometry>
+                <!-- 材料颜色 -->
+                <material name="yellow">
+                    <color rgba="1.0 1.0 0.0 0.8"/>
+                </material>
+            </collision>
         </link>
         <!-- 机器人的关节，用于组合机器人的部件 -->
@@ -22,4 +33,5 @@
             <origin xyz="${xyz}" rpy="0.0 0.0 0.0"/>
         </joint>
+        <xacro:sphere_inertia m="0.05" r="0.016" />
     </xacro:macro>
 </robot>

File: src/wmq_description/urdf/wmqbot/actuator/wheel.urdf.xacro (robot description, xacro)
@@ -1,4 +1,5 @@
 <?xml version="1.0"?>
 <robot xmlns:xacro="http://www.ros.org/wiki/xacro">
+    <xacro:include filename="$(find wmq_description)/urdf/wmqbot/common_inertia.xacro" />
     <xacro:macro name="wheel_xacro" params="wheel_name xyz">
         <!-- 机器人的身体部分 -->
@@ -14,4 +15,14 @@
                 </material>
             </visual>
+            <collision>
+                <origin xyz="0.0 0.0 0.0" rpy="1.57079 0.0 0.0"/>
+                <geometry>
+                    <cylinder radius="0.032" length="0.04"/>
+                </geometry>
+                <material name="yellow">
+                    <color rgba="1.0 1.0 0.0 0.8"/>
+                </material>
+            </collision>
+            <xacro:cylinder_inertia m="0.05" r="0.032" h="0.04" />
         </link>
         <!-- 机器人的关节，用于组合机器人的部件 -->

File: src/wmq_description/urdf/wmqbot/base.urdf.xacro (robot description, xacro)
@@ -1,5 +1,7 @@
 <?xml version="1.0"?>
 <robot xmlns:xacro="http://www.ros.org/wiki/xacro">
+    <xacro:include filename="$(find wmq_description)/urdf/wmqbot/common_inertia.xacro" />
     <xacro:macro name="base_xacro" params="length radius">
+        <link name="base_footprint" />
         <!-- 机器人的身体部分 -->
         <link name="base_link">
@@ -10,9 +12,24 @@
                     <cylinder radius="${radius}" length="${length}"/>
                 </geometry>
-                <material name="black">
+                <material name="white">
                     <color rgba="1.0 1.0 1.0 0.5"/>
                 </material>
             </visual>
+            <collision>
+                <origin xyz="0.0 0.0 0.0" rpy="0.0 0.0 0.0"/>
+                <geometry>
+                    <cylinder radius="${radius}" length="${length}"/>
+                </geometry>
+                <material name="white">
+                    <color rgba="1.0 1.0 1.0 0.5"/>
+                </material>
+            </collision>
+            <xacro:cylinder_inertia m="1.0" r="${radius}" h="${length}" />
         </link>
+        <joint name="joint_name" type="fixed">
+            <origin xyz="0.0 0.0 ${length/2.0+0.032-0.01}" rpy="0.0 0.0 0.0"/>
+            <parent link="base_footprint"/>
+            <child link="base_link"/>
+        </joint>
     </xacro:macro>
 </robot>

File: src/wmq_description/urdf/wmqbot/sensor/camera.urdf.xacro (robot description, xacro)
@@ -1,4 +1,5 @@
 <?xml version="1.0"?>
 <robot xmlns:xacro="http://www.ros.org/wiki/xacro">
+    <xacro:include filename="$(find wmq_description)/urdf/wmqbot/common_inertia.xacro" />
     <xacro:macro name="camera_xacro" params="xyz">
         <!-- 机器人的相机部件，惯性测量传感器 -->
@@ -13,4 +14,15 @@
                 </material>
             </visual>
+            <collision>
+                <origin xyz="0.0 0.0 0.0" rpy="0.0 0.0 0.0"/>
+                <geometry>
+                    <box size="0.02 0.10 0.02"/>
+                </geometry>
+                <material name="black">
+                    <color rgba="1.0 1.0 1.0 0.5"/>
+                </material>
+            </collision>
+            <!-- 加入重心和偏移 -->
+            <xacro:box_inertia m="0.1" w="0.02" h="0.10" d="0.02" />
         </link>
         <!-- 机器人的关节，用于组合机器人的部件 -->

File: src/wmq_description/urdf/wmqbot/sensor/imu.urdf.xacro (robot description, xacro)
@@ -1,4 +1,5 @@
 <?xml version="1.0"?>
 <robot xmlns:xacro="http://www.ros.org/wiki/xacro">
+    <xacro:include filename="$(find wmq_description)/urdf/wmqbot/common_inertia.xacro" />
     <xacro:macro name="imu_xacro" params="xyz">
         <!-- 机器人的IMU部件，惯性测量传感器 -->
@@ -13,4 +14,14 @@
                 </material>
             </visual>
+            <collision>
+                <origin xyz="0.0 0.0 0.0" rpy="0.0 0.0 0.0"/>
+                <geometry>
+                    <box size="0.02 0.02 0.02"/>
+                </geometry>
+                <material name="black">
+                    <color rgba="0.0 0.0 0.0 0.5"/>
+                </material>
+            </collision>
+            <xacro:box_inertia m="0.05" w="0.02" h="0.02" d="0.02"/>
         </link>
         <!-- 机器人的关节，用于组合机器人的部件 -->

File: src/wmq_description/urdf/wmqbot/sensor/laser.urdf.xacro (robot description, xacro)
@@ -1,4 +1,5 @@
 <?xml version="1.0"?>
 <robot xmlns:xacro="http://www.ros.org/wiki/xacro">
+    <xacro:include filename="$(find wmq_description)/urdf/wmqbot/common_inertia.xacro" />
     <xacro:macro name="laser_xacro" params="xyz">
         <!-- 雷达支撑杆 -->
@@ -14,4 +15,14 @@
                 </material>
             </visual>
+            <collision>
+                <origin xyz="0.0 0.0 0.0" rpy="0.0 0.0 0.0"/>
+                <geometry>
+                    <cylinder radius="0.01" length="0.10"/>
+                </geometry>
+                <material name="black">
+                    <color rgba="0.0 0.0 0.0 1.0"/>
+                </material>
+            </collision>
+            <xacro:cylinder_inertia m="0.05" r="0.01" h="0.10" />
         </link>
         <!-- 雷达 -->
@@ -28,4 +39,15 @@
                 </material>
             </visual>
+            <collision>
+                <origin xyz="0.0 0.0 0.0" rpy="0.0 0.0 0.0"/>
+                <geometry>
+                    <cylinder radius="0.02" length="0.02"/>
+                </geometry>
+                <!-- 材料颜色 -->
+                <material name="black">
+                    <color rgba="0.0 0.0 0.0 1.0"/>
+                </material>
+            </collision>
+            <xacro:cylinder_inertia m="0.10" r="0.02" h="0.02" />
         </link>
         <!-- 机器人的关节，用于组合机器人的部件 -->

Commit message: 关节状态发布工具有bug

File: src/wmq_description/urdf/wmqbot/actuator/caster.urdf.xacro (robot description, xacro)
@@ -26,4 +26,5 @@
                 </material>
             </collision>
+        <xacro:sphere_inertia m="0.05" r="0.016" />
         </link>
         <!-- 机器人的关节，用于组合机器人的部件 -->
@@ -33,5 +34,14 @@
             <origin xyz="${xyz}" rpy="0.0 0.0 0.0"/>
         </joint>
-        <xacro:sphere_inertia m="0.05" r="0.016" />
+        <gazebo reference="${caster_name}_link">
+            <!-- 切向摩擦系数 -->
+            <mu1 value="0.0"/>
+            <!-- 法向摩擦系数 -->
+            <mu2 value="0.0"/>
+            <!-- 刚度系数 -->
+            <kp value="1000000000.0"/>
+            <!-- 阻尼系数 -->
+            <kd value="1.0"/>
+        </gazebo>
     </xacro:macro>
 </robot>

File: src/wmq_description/urdf/wmqbot/actuator/wheel.urdf.xacro (robot description, xacro)
@@ -33,4 +33,14 @@
             <axis xyz="0 1 0"/>
         </joint>
+        <gazebo reference="${wheel_name}_link">
+            <!-- 切向摩擦系数 -->
+            <mu1 value="20.0"/>
+            <!-- 法向摩擦系数 -->
+            <mu2 value="20.0"/>
+            <!-- 刚度系数 -->
+            <kp value="1000000000.0"/>
+            <!-- 阻尼系数 -->
+            <kd value="1.0"/>
+        </gazebo>
     </xacro:macro>
 </robot>

File: src/wmq_description/urdf/wmqbot/sensor/camera.urdf.xacro (robot description, xacro)
@@ -26,4 +26,5 @@
             <xacro:box_inertia m="0.1" w="0.02" h="0.10" d="0.02" />
         </link>
+        <link name="camera_optical_link"></link>
         <!-- 机器人的关节，用于组合机器人的部件 -->
         <joint name="camera_joint" type="fixed">
@@ -32,4 +33,9 @@
             <origin xyz="${xyz}" rpy="0.0 0.0 0.0"/>
         </joint>
+        <joint name="camera_optical_joint" type="fixed">
+            <parent link="camera_link"/>
+            <child link="camera_optical_link"/>
+            <origin xyz="0 0 0" rpy="${-pi/2} 0.0 ${-pi/2}"/>
+        </joint>
     </xacro:macro>
 </robot>

File: src/wmq_description/urdf/wmqbot/sensor/laser.urdf.xacro (robot description, xacro)
@@ -62,4 +62,10 @@
             <origin xyz="${xyz}" rpy="0.0 0.0 0.0"/>
         </joint>
+        <gazebo reference="laser_cylinder_link">
+            <material>Gazebo/Black</material>
+        </gazebo>
+        <gazebo reference="laser_link">
+            <material>Gazebo/Black</material>
+        </gazebo>
     </xacro:macro>
 </robot>

File: src/wmq_description/urdf/wmqbot/wmqbot.urdf.xacro (robot description, xacro)
@@ -10,4 +10,8 @@
 <xacro:include filename="$(find wmq_description)/urdf/wmqbot/actuator/wheel.urdf.xacro"/>
 <xacro:include filename="$(find wmq_description)/urdf/wmqbot/actuator/caster.urdf.xacro"/>
+<!-- 插件 -->
+<!-- <xacro:include filename="$(find wmq_description)/urdf/wmqbot/plugins/gazebo_control_plugin.xacro"/> -->
+<xacro:include filename="$(find wmq_description)/urdf/wmqbot/plugins/gazebo_sensor_plugin.xacro"/>
+<xacro:include filename="$(find wmq_description)/urdf/wmqbot/wmqbot.ros2_control.xacro"/>
 <xacro:base_xacro length="0.12" radius="0.10"/>
 <xacro:imu_xacro xyz="0.0 0.0 0.02"/>
@@ -18,3 +22,6 @@
 <xacro:caster_xacro caster_name="front_wheel" xyz="0.08 0.0 -0.076"/>
 <xacro:caster_xacro caster_name="back_wheel" xyz="-0.08 0.0 -0.076"/>
+<!-- <xacro:gazebo_control_plugin /> -->
+<xacro:gazebo_sensor_plugin />
+<xacro:wmqbot_ros2_control />
 </robot>
